Commit message: homework_finito_davvero

File: arm_description/urdf/arm.urdf.xacro (robot description, xacro)
@@ -10,4 +10,10 @@
     <color rgba="1 1 1 1"/>
   </material>
+  <link name="world"/>
+  <joint name="base_link_joint" type="fixed">
+    <parent link="world"/>
+    <child link="base_link"/>
+    <origin rpy="0 0 0 0" xyz="0 0 0 0"/>
+  </joint>
  <link name="base_link">
     <visual>
